File: PCB/EPS Kicad Design/EPS_KiCad_Design/3V3.kicad_sch (KiCad schematic)
At the start: 7 parts, among them IC3 LM2675M-3.3_NOPB, J3 Conn_01x02_Pin

Commit message: Actualizacion del PCB en Kicad
Parts:
- removed D6: D_Zener, symbol Device:D_Zener
- removed J3: Conn_01x02_Pin, symbol Connector:Conn_01x02_Pin
- added C20: 0.1uF, Capacitor_SMD:C_0805_2012Metric_Pad1.18x1.45mm_HandSolder, symbol Device:C
- added D14: MBRS340, Diode_SMD:D_SMC, symbol Diode:MBRS340
- added IC8: INA226AIDGST, INA226AIDGST_Footprint:SOP50P490X110-10N, symbol INA226AIDGST:INA226AIDGST
- added J3: Conn_01x02, symbol Connector_Generic:Conn_01x02
- added R20: 0.05, Resistor_SMD:R_0805_2012Metric_Pad1.20x1.40mm_HandSolder, symbol Device:R
- C4: value C -> 22uF; footprint (none) -> Capacitor_SMD:C_0805_2012Metric_Pad1.18x1.45mm_HandSolder
- C5: value C -> 0.01uF; footprint (none) -> Capacitor_SMD:C_0805_2012Metric_Pad1.18x1.45mm_HandSolder
- C6: value C -> 47uF; footprint (none) -> Capacitor_SMD:C_0805_2012Metric_Pad1.18x1.45mm_HandSolder
- L2: value L -> 68uH
Connections:
- net 3V3: now also C20.1, IC8.2 (A0), IC8.6 (VS), IC8.8 (VBUS), IC8.9 (IN-), J3.1 (Pin_1), R20.1; no longer C6.2, IC3.4 (FB), L2.1
- net GND: now also C20.2, D14.2 (A), IC8.1 (A1), IC8.7 (GND), J3.2 (Pin_2)
- net at C5.1, IC3.8 (VSW), L2.2: now also D14.1 (K)
- net Vsystem: now reaches C4.1, IC3.7 (VIN)
- net EN_3V3 renamed GPIO
- new net ALERT2: IC8.3 (ALERT)
- new net IN1+: C6.2, IC3.4 (FB), IC8.10 (IN+), L2.1, R20.2
- new net SCL2: IC8.5 (SCL)
- new net SDA2: IC8.4 (SDA)
Other:
- note added: "Monitor de voltaje, corriente y potencia"
- note added: "Salida al sistema"
- note removed: "V_REGULATOR-3V3"
