File: PCB/EPS Kicad Design/EPS_KiCad_Design/EPS_KiCad_Design.kicad_sch (KiCad schematic)
At the start: 0 parts

Commit message: Actualizacion del PCB en Kicad
Other:
- removed sheet MPPT
- added sheet MCU (MCU.kicad_sch)
- added sheet MPPT + BATTERY CHARGER (MPPT_BatteryChager.kicad_sch)
- note added: "- Agregar un deployment switch (investigar cómo se hace)"
- note added: "- Agregar una salida no regulada con un OCP"
- note added: "- Agregarle un sensor de temperatura a la batería (no puede bajar a 0°)"
- note added: "OBSERVACIONES"
Changed lines of the file:
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@@
 		(comment 4 "By: Danis González, Tobias Decoud")
 	)
+	(text "OBSERVACIONES"
+		(exclude_from_sim no)
+		(at 245.11 18.034 0)
+		(effects
+			(font
+				(size 1.27 1.27)
+				(thickness 0.254)
+				(bold yes)
+				(italic yes)
+			)
+		)
+	)
+	(text "- Agregar un deployment switch (investigar cómo se hace)"
+		(exclude_from_sim no)
+		(at 239.014 26.67 0)
+		(effects
+			(font
+				(size 1.27 1.27)
+			)
+		)
+	)
+	(text "- Agregarle un sensor de temperatura a la batería (no puede bajar a 0°)"
+		(exclude_from_sim no)
+		(at 246.634 22.606 0)
+		(effects
+			(font
+				(size 1.27 1.27)
+			)
+		)
+	)
+	(text "- Agregar una salida no regulada con un OCP"
+		(exclude_from_sim no)
+		(at 232.918 31.242 0)
+		(effects
+			(font
+				(size 1.27 1.27)
+			)
+		)
+	)
 	(sheet
-		(at 186.69 78.74)
-		(size 33.02 30.48)
+		(at 198.12 81.28)
+		(size 46.99 31.75)
 		(exclude_from_sim no)
 		(in_bom yes)
@@
 			(color 0 0 0 0.0000)
 		)
-		(property "Sheetname" "MPPT"
-			(at 186.69 78.0284 0)
+		(property "Sheetname" "MPPT + BATTERY CHARGER"
+			(at 198.12 80.5684 0)
 			(effects
 				(font
@@
 			)
 		)
-		(property "Sheetfile" "MPPT.kicad_sch"
-			(at 186.69 109.8046 0)
+		(property "Sheetfile" "MPPT_BatteryChager.kicad_sch"
+			(at 198.12 113.6146 0)
 			(effects
 				(font
@@
 			(project "EPS_KiCad_Design"
 				(path "/86c6bf32-0fdc-4559-bb3e-0b6f31730fee"
-					(page "2")
+					(page "7")
 				)
 			)
@@
 	)
 	(sheet
-		(at 111.76 77.47)
-		(size 40.64 33.02)
+		(at 140.97 80.01)
+		(size 45.72 33.02)
 		(exclude_from_sim no)
 		(in_bom yes)
@@
 		)
 		(property "Sheetname" "Voltage Converter"
-			(at 111.76 76.7584 0)
+			(at 140.97 79.2984 0)
 			(effects
 				(font
@@
 		)
 		(property "Sheetfile" "VoltageConverter.kicad_sch"
-			(at 111.76 111.0746 0)
+			(at 140.97 113.6146 0)
 			(effects
 				(font
@@
 				)
 			)
+		)
+	)
+	(sheet
+		(at 82.55 80.01)
+		(size 44.45 33.02)
+		(exclude_from_sim no)
+		(in_bom yes)
+		(on_board yes)
+		(dnp no)
+		(fields_autoplaced yes)
+		(stroke
+			(width 0.1524)
+			(type solid)
+		)
+		(fill
+			(color 0 0 0 0.0000)
+		)
+		(property "Sheetname" "MCU"
+			(at 82.55 79.2984 0)
+			(effects
+				(font
+					(size 1.27 1.27)
+				)
+				(justify left bottom)
+			)
+		)
+		(property "Sheetfile" "MCU.kicad_sch"
+			(at 82.55 113.6146 0)
+			(effects
+				(font
+					(size 1.27 1.27)
+				)
+				(justify left top)
+			)
+		)
+		(instances
+			(project "EPS_KiCad_Design"
+				(path "/86c6bf32-0fdc-4559-bb3e-0b6f31730fee"
+					(page "6")
+				)
+			)
