File: PCB/EPS Kicad Design/EPS_KiCad_Design/MPPT.kicad_sch (KiCad schematic)
At the start: 23 parts, among them IC1 LT3652IMSE#PBF, IC2 INA138NA_250, J1 Conn_01x02_Pin, J2 Conn_01x01_Pin

Commit message: Actualizacion del PCB en Kicad
Other:
- note removed: "- El current & power monitor es diferente al usado en la tesis de grado, esto debido a su disponinilidad"
- note removed: "- Esquema inspirado en una tesis de grado de la Univesidad Politécnica de Catalunya"
- note removed: "- Falta dimensionar acorde a la batería y los paneles solares."
Changed lines of the file:
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@@
 		(comment 4 "By: Danis González, Tobias Decoud")
-	)
-	(text "- Esquema inspirado en una tesis de grado de la Univesidad Politécnica de Catalunya"
-		(exclude_from_sim no)
-		(at 241.554 30.226 0)
-		(effects
-			(font
-				(size 1.27 1.27)
-			)
-		)
-	)
-	(text "- Falta dimensionar acorde a la batería y los paneles solares. "
-		(exclude_from_sim no)
-		(at 230.632 27.432 0)
-		(effects
-			(font
-				(size 1.27 1.27)
-			)
-		)
-	)
-	(text "- El current & power monitor es diferente al usado en la tesis de grado, esto \ndebido a su disponinilidad"
-		(exclude_from_sim no)
-		(at 237.998 34.29 0)
-		(effects
-			(font
-				(size 1.27 1.27)
-			)
-		)
 	)
 	(junction
@@
 		(on_board yes)
 		(dnp no)
-		(fields_autoplaced yes)
 		(property "Reference" "IC1"
 			(at 128.27 72.39 0)
@@
 		)
 		(property "Footprint" "LM3652IMSE_Footprint:SOP65P490X110-13N"
-			(at 142.24 174.93 0)
+			(at 107.442 68.58 0)
 			(effects
 				(font
@@
 		)
 		(property "Footprint" "INA138NA_Footprint:SOT95P280X145-5N"
-			(at 233.68 181.28 0)
-			(effects
-				(font
+			(at 233.426 92.964 0)
+			(effects
+				(font
