File: PCB/EPS Kicad Design/EPS_KiCad_Design/VoltageConverter.kicad_sch (KiCad schematic)
At the start: 0 parts

Commit message: Actualizacion del PCB en Kicad
Other:
- sheet 3V3 renamed 3V3 Principal + OCP
- sheet 5V renamed 5V + OCP
- removed sheet 12 V
- added sheet 3V3 Misiones + OCP (3V3MisionesWithOCP.kicad_sch)
- sheet 3V3 Principal + OCP: file 3V3.kicad_sch -> 3V3PrincipalwithOCP.kicad_sch
- sheet 5V + OCP: file 5V.kicad_sch -> 5VwithOCP.kicad_sch
- note added: "- Cada voltage converter tiene su propio encapsulado dedicado (Preguntar si es la forma correcta)"
- note added: "OBSERVACIONES"
- note removed: "Cada voltage converter tiene su propio encapsulado dedicado (Preguntar si es la forma correcta)"
Changed lines of the file:
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@@
 		(comment 4 "By: Danis González, Tobias Decoud")
 	)
-	(text "Cada voltage converter tiene su propio encapsulado dedicado\n(Preguntar si es la forma correcta)"
+	(rectangle
+		(start 218.44 13.97)
+		(end 284.48 29.21)
+		(stroke
+			(width 0)
+			(type default)
+		)
+		(fill
+			(type none)
+		)
+	)
+	(text "- Cada voltage converter tiene su propio encapsulado dedicado\n(Preguntar si es la forma correcta)"
 		(exclude_from_sim no)
-		(at 251.206 18.542 0)
+		(at 251.46 22.098 0)
 		(effects
 			(font
@@
 		)
 	)
+	(text "OBSERVACIONES"
+		(exclude_from_sim no)
+		(at 252.73 17.78 0)
+		(effects
+			(font
+				(size 1.27 1.27)
+				(thickness 0.254)
+				(bold yes)
+				(italic yes)
+			)
+		)
+	)
 	(sheet
-		(at 111.76 77.47)
-		(size 50.8 34.29)
+		(at 177.8 76.2)
+		(size 46.99 34.29)
 		(exclude_from_sim no)
 		(in_bom yes)
@@
 			(color 0 0 0 0.0000)
 		)
-		(property "Sheetname" "5V"
-			(at 111.76 76.7584 0)
+		(property "Sheetname" "5V + OCP"
+			(at 177.8 75.4884 0)
 			(effects
 				(font
@@
 			)
 		)
-		(property "Sheetfile" "5V.kicad_sch"
-			(at 111.76 112.3446 0)
+		(property "Sheetfile" "5VwithOCP.kicad_sch"
+			(at 177.8 111.0746 0)
 			(effects
 				(font
@@
 	)
 	(sheet
-		(at 184.15 78.74)
-		(size 50.8 34.29)
+		(at 55.88 76.2)
+		(size 43.18 35.56)
 		(exclude_from_sim no)
 		(in_bom yes)
@@
 			(color 0 0 0 0.0000)
 		)
-		(property "Sheetname" "12 V"
-			(at 184.15 78.0284 0)
+		(property "Sheetname" "3V3 Misiones + OCP"
+			(at 55.88 75.4884 0)
 			(effects
 				(font
@@
 			)
 		)
-		(property "Sheetfile" "12V.kicad_sch"
-			(at 184.15 113.6146 0)
+		(property "Sheetfile" "3V3MisionesWithOCP.kicad_sch"
+			(at 55.88 112.3446 0)
 			(effects
 				(font
@@
 			(project "EPS_KiCad_Design"
 				(path "/86c6bf32-0fdc-4559-bb3e-0b6f31730fee/ac23d778-e7c7-4599-a635-b854b8369412"
-					(page "6")
+					(page "9")
 				)
 			)
@@
 	)
 	(sheet
-		(at 46.99 77.47)
+		(at 113.03 76.2)
 		(size 45.72 34.29)
 		(exclude_from_sim no)
@@
 			(color 0 0 0 0.0000)
 		)
-		(property "Sheetname" "3V3"
-			(at 46.99 76.7584 0)
+		(property "Sheetname" "3V3 Principal + OCP"
+			(at 113.03 75.4884 0)
 			(effects
 				(font
@@
 			)
 		)
-		(property "Sheetfile" "3V3.kicad_sch"
-			(at 46.99 112.3446 0)
+		(property "Sheetfile" "3V3PrincipalwithOCP.kicad_sch"
+			(at 113.03 111.0746 0)
 			(effects
 				(font
