File: PCB/EPS_KiCad_Design ruteo tobi/EPS_KiCad_Design/5VwithOCP.kicad_sch (KiCad schematic)
At the start: 18 parts, among them IC3 INA226AIDGST, IC4 TPS2553QDBVRQ1, IC5 AP63205WU-7

Commit message: pcb tobi
Connections:
- net SW: now reaches C11.2, IC5.5 (SW), L2.1
- net ILIM: now reaches IC4.5 (ILIM), R8.1
Changed lines of the file:
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@@
+		)
+	)
+	(label "SW"
+		(at 101.6 146.05 270)
+		(effects
+			(font
+				(size 1.27 1.27)
+			)
+			(justify right bottom)
 		)
 	)
@@
 		(effects
 			(font
+				(size 1.27 1.27)
+			)
+			(justify left bottom)
+		)
+	)
+	(label "ILIM"
+		(at 106.68 52.07 0)
+		(effects
+			(font
