File: PCB/EPS_KiCad_Design ruteo tobi/EPS_KiCad_Design/MPPT_BatteryChager.kicad_sch (KiCad schematic)
At the start: 48 parts, among them IC7 LT3652IMSE#PBF, IC8 INA226AIDGST, IC9 TPS25921ADR, J3 501568-0207, J4 Conn_01x04, J5 Conn_01x04, J6 501568-0207, J7 501568-0207, J8 Conn_01x04, J9 Conn_01x04

Commit message: pcb tobi
Parts:
- removed J3, J6: 501568-0207, 501568-0207_Footprint:5015680207, symbol 501568-0207:501568-0207
- added J10, J3: Conn_01x04, 62000411722_Footprint:62000411722, symbol Connector_Generic:Conn_01x04
- D2, D3, D4, D5: footprint Diode_SMD:D_SMC -> PMEG:SODFL3517X110N
Connections:
- net GND: now also J9.1 (Pin_1), J9.2 (Pin_2); no longer J9.3 (Pin_3), J9.4 (Pin_4)
- net IN-: now also J3.3 (Pin_3), J3.4 (Pin_4)
- net Vin: now also J10.3 (Pin_3), J10.4 (Pin_4)
- net Vsystem: now also J3.1 (Pin_1), J3.2 (Pin_2)
- net 2J3: now reaches C33.1, D5.2 (A), R16.1, SD15-01FTG1.1 (K)
- net 2J3: now also J10.1 (Pin_1), J10.2 (Pin_2)
- net SW: now reaches C29.1, D2.1 (K), IC7.12 (SW), L3.1
- net VIN: now reaches C32.1, D5.1 (K), D7.2 (A), D8.2 (A), IC7.1 (VIN)
- net BOOST: now reaches C29.2, D6.1 (K), IC7.11 (BOOST)
- net OUT: now reaches C37.1, IC9.5 (OUT), R29.1, SD12-01FTG2.1 (K)
- net OUT: now also J9.3 (Pin_3), J9.4 (Pin_4); no longer J9.1 (Pin_1), J9.2 (Pin_2)
