File: PCB/EPS_KiCad_Design ruteo tobi/EPS_KiCad_Design/EPS_KiCad_Design.kicad_pcb (KiCad board)
At the start: 4 copper layers, 90 x 90.2 mm, 133 parts, among them IC1 INA226AIDGST, IC10 TPS2553QDBVRQ1, IC11 INA226AIDGST, IC2 TPS2553QDBVRQ1, IC3 INA226AIDGST, IC4 TPS2553QDBVRQ1, IC5 AP63205WU-7, IC6 STM32L433CBT7, IC7 LT3652IMSE#PBF, IC8 INA226AIDGST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

Commit message: Correcciones MCU ruteo
Routing:
- net 3V3_2: track 68.4 -> 91.8 mm
- net GND: vias 241 -> 242
Changed lines of the file:
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@@
 		)
 		(embedded_fonts no)
-		(model "FTSH-107-01-L-D-K.stp"
+		(model "C:/Users/tobia/Downloads/EPS Kicad Design (1)/EPS Kicad Design/EPS Kicad Design/EPS_KiCad_Design/Library/FTSH-107-01-L-D-K/3D/FTSH-107-01-L-D-K.stp"
 			(offset
-				(xyz 3.769999924 0.6899999873 0.4499999813)
+				(xyz 3.77 0.69 -0.05)
 			)
 			(scale
@@
 			(at -3.5 0 90)
 			(layer "F.SilkS")
+			(hide yes)
 			(effects
 				(font
@@
 	)
 	(via
+		(at 121.5 75)
+		(size 0.6)
+		(drill 0.3)
+		(layers "F.Cu" "B.Cu")
+		(free yes)
+		(net 14)
+	)
+	(via
 		(at 142.565 88.10875)
 		(size 0.6)
@@
 	)
 	(segment
-		(start 138.25 106.957786)
-		(end 138.25 112.85)
-		(width 0.6)
-		(layer "In2.Cu")
-		(net 15)
-	)
-	(segment
-		(start 138.25 87.25)
-		(end 138.25 106.142214)
+		(start 138.174 87.326)
+		(end 138.174 112.926)
 		(width 0.6)
 		(layer "In2.Cu")
@@
 	(segment
 		(start 139.2 86.3)
-		(end 138.25 87.25)
-		(width 0.6)
-		(layer "In2.Cu")
-		(net 15)
-	)
-	(segment
-		(start 138.25 106.142214)
-		(end 138.174 106.218214)
+		(end 138.174 87.326)
 		(width 0.6)
 		(layer "In2.Cu")
@@
 	)
 	(segment
-		(start 138.174 106.218214)
-		(end 138.174 106.881786)
-		(width 0.6)
-		(layer "In2.Cu")
-		(net 15)
-	)
-	(segment
-		(start 138.174 106.881786)
-		(end 138.25 106.957786)
-		(width 0.6)
-		(layer "In2.Cu")
-		(net 15)
-	)
-	(segment
-		(start 138.25 112.85)
+		(start 138.174 112.926)
 		(end 137.2 113.9)
 		(width 0.6)
@@
 	)
 	(segment
-		(start 124.335 77.035)
-		(end 124.7 77.4)
-		(width 0.2)
+		(start 123.2 76.3)
+		(end 123.2 77.035)
+		(width 0.6)
 		(layer "F.Cu")
 		(net 16)
@@
 	)
 	(segment
+		(start 122.1 75.6)
+		(end 122.5 75.6)
+		(width 0.6)
+		(layer "F.Cu")
+		(net 16)
+	)
+	(segment
 		(start 168.12 85.72)
 		(end 166.78 85.72)
@@
 	)
 	(segment
-		(start 123.2 77.035)
-		(end 124.335 77.035)
-		(width 0.2)
+		(start 122.5 75.6)
+		(end 123.2 76.3)
+		(width 0.6)
 		(layer "F.Cu")
 		(net 16)
@@
 	)
 	(via
-		(at 124.7 77.4)
-		(size 0.7)
+		(at 122.1 75.6)
+		(size 0.6)
 		(drill 0.3)
 		(layers "F.Cu" "B.Cu")
@@
 	)
 	(segment
-		(start 137.35 94.35)
-		(end 137.35 92.9)
-		(width 0.2)
+		(start 122.1 90.8)
+		(end 125.65 94.35)
+		(width 0.6)
 		(layer "In2.Cu")
 		(net 16)
 	)
 	(segment
-		(start 137.35 92.9)
-		(end 124.7 80.25)
-		(width 0.2)
+		(start 125.65 94.35)
+		(end 137.35 94.35)
+		(width 0.6)
 		(layer "In2.Cu")
 		(net 16)
 	)
 	(segment
-		(start 158.9 84.1)
-		(end 160.95 86.15)
-		(width 0.2)
+		(start 146.567214 73.7)
+		(end 159.017214 86.15)
+		(width 0.6)
 		(layer "In2.Cu")
 		(net 16)
 	)
 	(segment
-		(start 140.15 84.1)
-		(end 158.9 84.1)
-		(width 0.2)
+		(start 122.1 75.6)
+		(end 122.1 90.8)
+		(width 0.6)
 		(layer "In2.Cu")
 		(net 16)
 	)
 	(segment
-		(start 137.35 92.9)
-		(end 137.35 86.9)
-		(width 0.2)
+		(start 124 73.7)
+		(end 146.567214 73.7)
+		(width 0.6)
 		(layer "In2.Cu")
 		(net 16)
 	)
 	(segment
-		(start 124.7 80.25)
-		(end 124.7 77.4)
-		(width 0.2)
+		(start 159.017214 86.15)
+		(end 160.95 86.15)
+		(width 0.6)
 		(layer "In2.Cu")
 		(net 16)
 	)
 	(segment
-		(start 137.35 86.9)
-		(end 140.15 84.1)
-		(width 0.2)
+		(start 122.1 75.6)
+		(end 124 73.7)
+		(width 0.6)
 		(layer "In2.Cu")
 		(net 16)
@@
 	)
 	(via
-		(at 130.8 97)
-		(size 0.6)
+		(at 131 97)
+		(size 0.7)
 		(drill 0.3)
 		(layers "F.Cu" "B.Cu")
@@
 	)
 	(segment
-		(start 130.8 97)
+		(start 130.8 96.8)
 		(end 130.8 96.75)
 		(width 0.2)
@@
 	)
 	(segment
-		(start 130.8 96.75)
-		(end 130.15 96.1)
+		(start 131 97)
+		(end 130.8 96.8)
 		(width 0.2)
 		(layer "In2.Cu")
@@
 	)
 	(segment
+		(start 130.8 96.75)
+		(end 130.15 96.1)
+		(width 0.2)
+		(layer "In2.Cu")
+		(net 22)
+	)
+	(segment
 		(start 125.45 96.1)
 		(end 123.9 94.55)
@@
 	)
 	(segment
-		(start 136.195 115.24)
-		(end 138.125 115.24)
+		(start 138.975 117.875)
+		(end 138.82 117.72)
 		(width 0.2)
 		(layer "F.Cu")
@@
 	)
 	(segment
-		(start 173.570831 118.351593)
-		(end 174.731238 119.512)
+		(start 136.195 115.24)
+		(end 138.125 115.24)
 		(width 0.2)
 		(layer "F.Cu")
@@
 	)
 	(segment
-		(start 138.975 117.875)
-		(end 138.82 117.72)
+		(start 173.570831 118.351593)
+		(end 174.731238 119.512)
 		(width 0.2)
 		(layer "F.Cu")
@@
 	)
 	(segment
-		(start 138.975 117.875)
-		(end 139.325 117.875)
+		(start 139.325 117.875)
+		(end 139.851 117.349)
 		(width 0.2)
 		(layer "In2.Cu")
@@
 	)
 	(segment
-		(start 153.672247 118.351593)
-		(end 173.570831 118.351593)
+		(start 152.669654 117.349)
+		(end 153.672247 118.351593)
 		(width 0.2)
 		(layer "In2.Cu")
@@
 	)
 	(segment
-		(start 152.669654 117.349)
-		(end 153.672247 118.351593)
+		(start 138.975 117.875)
+		(end 139.325 117.875)
 		(width 0.2)
 		(layer "In2.Cu")
@@
 	)
 	(segment
-		(start 139.325 117.875)
-		(end 139.851 117.349)
+		(start 153.672247 118.351593)
+		(end 173.570831 118.351593)
 		(width 0.2)
 		(layer "In2.Cu")
@@
 			"2c2b062a-b2b3-4ee9-85a2-bf9d8af9ab64" "32d6b5a0-03eb-4269-84d0-69514add3b08"
 			"35f5caa2-aac8-46bb-8a11-19497ad65581" "3af609cd-d4ae-41d7-9300-25bc8f08d530"
-			"3b09522c-e3b9-4279-8fce-4fc0c7d76b1a" "46552812-2f8f-4e24-8fb0-fa7be8f73b60"
-			"4698bc4f-d8ae-4a72-88ea-78ab5dd542c8" "46e0b36c-c088-4128-8487-8c732b78b328"
-			"4d66c90b-31e3-441d-86ca-dd21741283a6" "509566ee-1e86-4f42-ac8d-0c23405521b1"
-			"5a3972a1-545b-468e-ac88-6d811f49efb9" "5b4d0602-455b-47e9-8acd-8bc37e941de9"
-			"5ef308b7-a69a-41ed-9ac2-1d185bea8ddc" "60911e9f-3d44-4772-b8b8-b16590a952ae"
-			"66b4df74-e0f4-4fe3-b93b-6710d2ef82e9" "6704dd6f-c179-471f-be75-65c3a86bae91"
-			"6ad5cdd7-fb6a-46a9-aa80-280897e154fe" "6f00a87c-82c5-489e-a3f1-ad20767c2897"
-			"7496d75c-f986-4536-b2e0-fd371eae3c8b" "757f1288-6889-4dcb-b02b-25f34d31379f"
-			"77bf2897-e2c4-4220-8880-0db278073702" "7cc82f12-473a-404c-bef4-733f458daeab"
+			"46552812-2f8f-4e24-8fb0-fa7be8f73b60" "4d66c90b-31e3-441d-86ca-dd21741283a6"
+			"5b4d0602-455b-47e9-8acd-8bc37e941de9" "66b4df74-e0f4-4fe3-b93b-6710d2ef82e9"
+			"6704dd6f-c179-471f-be75-65c3a86bae91" "6ad5cdd7-fb6a-46a9-aa80-280897e154fe"
+			"6f00a87c-82c5-489e-a3f1-ad20767c2897" "7496d75c-f986-4536-b2e0-fd371eae3c8b"
+			"757f1288-6889-4dcb-b02b-25f34d31379f" "77bf2897-e2c4-4220-8880-0db278073702"
 			"82a5552a-8293-4e81-bbf4-07332a9ac419" "88876f19-8756-4372-8cac-0ec171e02209"
-			"8bff1752-c588-43b4-bbde-f47f6a2690b0" "8f3a95fe-8e4e-4235-be4a-99136b2687bf"
+			"8bff1752-c588-43b4-bbde-f47f6a2690b0" "9609b3ae-dbd6-49f6-83fc-c4881f3a1ac6"
 			"9e09712c-3f55-4ac3-8df4-923e149b7ed7" "9f7a25c8-637e-431e-91d6-c6805bed8244"
 			"a345f069-f284-47dd-9674-0044805ab73f" "a6178f8e-9587-4b87-8eb7-f759fed35891"
 			"aa099165-8a80-4ea6-896f-c93ae2e59488" "aac96920-5fa2-4061-b87c-fc06c307596b"
-			"afb9efb4-6f12-40c2-88cd-9f28558184dd" "bb20da57-fa69-4618-a401-f1213e73a4cc"
-			"c193dbdf-7a8f-4466-b83e-5230dc4539db" "c5087ba9-5f25-466d-beb7-af6bf17539de"
-			"c92d41fa-f27e-43dc-b4b5-87e7503bd0d2" "c95f9a0c-06c1-402c-9a67-ec4c89e969a1"
-			"cfaf2def-8399-4a92-a284-dd398f758917" "cfc57d06-7da5-4acf-ac7e-b5e12e6b62c5"
-			"d1f96a26-112f-497f-91e7-0e2c8f5b08e2" "d2c509b1-b3a8-435f-8084-171b6c0536d2"
-			"d852d3ce-fa8e-4d88-a7e5-bbd246105690" "e4fe2c6a-7bec-4b2c-92ec-ec724df715d8"
-			"f860916d-3c82-42c7-9004-221b3291a78c" "f9c856fd-2817-49a1-aed3-a8902f2e3d7d"
-			"ff73016c-a567-4195-8520-b240b5b45ee7"
+			"bb20da57-fa69-4618-a401-f1213e73a4cc" "c193dbdf-7a8f-4466-b83e-5230dc4539db"
+			"c95f9a0c-06c1-402c-9a67-ec4c89e969a1" "cb0219e1-0884-4c67-b679-1f42838dc0ea"
+			"cc01be6f-57ed-401b-aaa8-56deaa8dc9ba" "d1f96a26-112f-497f-91e7-0e2c8f5b08e2"
+			"d2c509b1-b3a8-435f-8084-171b6c0536d2" "d852d3ce-fa8e-4d88-a7e5-bbd246105690"
+			"e4fe2c6a-7bec-4b2c-92ec-ec724df715d8" "f7fbc15b-d2a6-4a4c-b1f4-5bcd74f74e2e"
+			"f9c856fd-2817-49a1-aed3-a8902f2e3d7d" "ff73016c-a567-4195-8520-b240b5b45ee7"
 		)
 	)
@@
 	)
 	(group ""
-		(members "10af0be8-4f90-40ef-a055-ece5ec01faff" "2972b692-cf6e-44d3-a4a5-dba2aa1ae555"
-			"2afe3086-7003-42cb-876a-61b162fe43f3" "2c54b120-fbeb-4924-ab7a-9d4e3238112a"
+		(members "10af0be8-4f90-40ef-a055-ece5ec01faff" "1b599d84-854c-41e4-a9bf-99bdc57952be"
+			"2972b692-cf6e-44d3-a4a5-dba2aa1ae555" "2afe3086-7003-42cb-876a-61b162fe43f3"
+			"2c54b120-fbeb-4924-ab7a-9d4e3238112a" "2fe15ccd-5528-4d57-98c7-ad29761bb398"
 			"3072a043-89d4-4446-8ad3-cf5feabf6e68" "3ee0addc-d812-404f-a938-d1b417fa6c09"
-			"4b5f78f5-f516-4eeb-bfdb-957901cc2800" "4e76fd0b-7eb7-490a-8fb3-2f2fa949279b"
-			"62811ce2-3539-4c98-aab3-60b3ad853782" "64f67280-b1d7-4152-9507-98e11ba6b3e3"
+			"4b5f78f5-f516-4eeb-bfdb-957901cc2800" "62811ce2-3539-4c98-aab3-60b3ad853782"
 			"6c1ff341-ef3f-4dce-9c9c-eead211bad09" "6ef52392-8809-48a9-a639-ddc3d01bc285"
 			"774b4c10-432b-4c2c-bf9d-1834bc9f489a" "77658e06-2e36-4c2a-a8da-610f299490d2"
-			"80830169-5f0c-4829-8151-a90b24aeeb2c" "84f8ba23-e680-41d1-a4ab-e375cd32ceca"
-			"9e1c8f42-ce4b-4b3b-a844-f19d569e08e1" "a534298b-d40b-46c9-96c1-71491df51e6b"
-			"b3e744f7-c078-4e75-8f77-c34c27a6ed89" "baafd113-30e2-43bb-ba08-6d6ccf037178"
+			"7f34ca46-cfc6-4187-b755-55caa72f7e67" "80830169-5f0c-4829-8151-a90b24aeeb2c"
+			"84f8ba23-e680-41d1-a4ab-e375cd32ceca" "9e1c8f42-ce4b-4b3b-a844-f19d569e08e1"
+			"a534298b-d40b-46c9-96c1-71491df51e6b" "baafd113-30e2-43bb-ba08-6d6ccf037178"
 			"c9ed9ae1-49e6-4635-b308-28ba9ab92d45" "cdada0dc-3e72-474b-ab61-1f051990450e"
 			"cf50b09b-f59b-45aa-87f8-0460bc0f20cd" "d07d1cd9-e83c-449f-8147-5501051456b4"
-			"dbcf1419-a2a1-4ad1-ac42-49c458d3bacf" "e75bef67-e118-4ab7-9e90-a17903169027"
-			"eb034991-ad5b-4658-b25c-1f7424faf62d" "ec3f9fa0-560b-420c-b3f6-e366f481388e"
-			"f127d90a-f94a-4f92-bbd4-144c3fcc3584" "fc681ca5-947f-41c9-9c3a-40a32c7771f7"
+			"d5b6b365-b883-4267-9124-087927e383dd" "dbcf1419-a2a1-4ad1-ac42-49c458d3bacf"
+			"e75bef67-e118-4ab7-9e90-a17903169027" "ec3f9fa0-560b-420c-b3f6-e366f481388e"
+			"f127d90a-f94a-4f92-bbd4-144c3fcc3584" "fab8cf9c-a207-491c-9253-be1ee5a54bda"
+			"fc681ca5-947f-41c9-9c3a-40a32c7771f7"
 		)
 	)

Commit message: RUTEO MCU
Routing:
- net SDA: track 6.27 -> 189.8 mm, vias 0 -> 6
- net SCL: track 3.36 -> 175.3 mm, vias 0 -> 6
- net ALERT: track 2.60 -> 165.5 mm, vias 0 -> 8
- net SDA OBC: track 0.00 -> 105.7 mm, vias 0 -> 1
- net SCL OBC: track 0.00 -> 95.6 mm, vias 0 -> 1
- net GPIO3: track 5.93 -> 89.1 mm, vias 0 -> 2
- net GPIO4: track 1.84 -> 84.9 mm, vias 0 -> 2
- net GPIO6: track 9.71 -> 86.7 mm, vias 0 -> 2
- net EN OBC: track 0.00 -> 75.2 mm, vias 0 -> 1
- net GPIO5: track 4.60 -> 78.9 mm, vias 0 -> 2
- net GPIO1: track 4.10 -> 69.2 mm, vias 0 -> 2
- net GPIO2: track 9.12 -> 67.2 mm, vias 0 -> 2
- net /MCU/PB3: track 0.00 -> 32.8 mm, vias 0 -> 2
- net /MCU/PA14: track 0.00 -> 31.3 mm, vias 0 -> 2
- net /MCU/PA13: track 0.00 -> 29.0 mm, vias 0 -> 2
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