File: PCB/EPS_KiCad_Design ruteo tobi/EPS_KiCad_Design/3V3MisionesWithOCP.kicad_sch (KiCad schematic)
At the start: 18 parts, among them IC10 TPS2553QDBVRQ1, IC11 INA226AIDGST

Commit message: pcb tobi
Connections:
- net SW: now reaches C41.2, D9.5 (SW), L4.1
- net ILIM: now reaches IC10.5 (ILIM), R33.1
Changed lines of the file:
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@@
+		)
+	)
+	(label "ILIM"
+		(at 95.25 53.34 0)
+		(effects
+			(font
+				(size 1.27 1.27)
+			)
+			(justify left bottom)
 		)
 	)
@@
 		)
 	)
+	(label "SW"
+		(at 93.98 138.43 270)
+		(effects
+			(font
+				(size 1.27 1.27)
+			)
+			(justify right bottom)
+		)
+	)

Commit message: Actualizacion del PCB
Parts:
- L4: footprint SRR4528A-3R9Y_Footprint:SRR4528A3R9Y -> ASPI:ASPI0628150MT1
Changed lines of the file:
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@@
 			)
 		)
-		(property "Footprint" "SRR4528A-3R9Y_Footprint:SRR4528A3R9Y"
+		(property "Footprint" "ASPI:ASPI0628150MT1"
 			(at 101.6 138.43 0)
 			(effects
