File: PCB/EPS_KiCad_Design ruteo tobi/EPS_KiCad_Design/3V3PrincipalwithOCP.kicad_sch (KiCad schematic)
At the start: 18 parts, among them IC1 INA226AIDGST, IC2 TPS2553QDBVRQ1

Commit message: Actualizacion del PCB
Parts:
- L1: footprint SRR4528A-3R9Y_Footprint:SRR4528A3R9Y -> ASPI:ASPI0628150MT1
Changed lines of the file:
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@@
 			)
 		)
-		(property "Footprint" "SRR4528A-3R9Y_Footprint:SRR4528A3R9Y"
+		(property "Footprint" "ASPI:ASPI0628150MT1"
 			(at 106.68 137.16 0)
 			(effects
