File: PCB/EPS_KiCad_Design ruteo tobi/EPS_KiCad_Design/EPS_KiCad_Design.kicad_sch (KiCad schematic)
At the start: 5 parts, among them J1 Conn_02x20_Counter_Clockwise

Commit message: cambios en el ruteo
Parts:
- removed H1, H2, H3, H4: MountingHole, MountingHole:MountingHole_3.2mm_M3_Pad_Via, symbol Mechanical:MountingHole
- added C46, C47, C48, C49: 100nF, Capacitor_SMD:C_0805_2012Metric_Pad1.18x1.45mm_HandSolder, symbol Device:C
- added H1, H2, H3, H4: MountingHole_Pad, MountingHole:MountingHole_3.2mm_M3_Pad_Via, symbol Mechanical:MountingHole_Pad
Connections:
- net GND: now also C46.2, C47.2, C48.1, C49.1
- new net: C48.2, H1.1
- new net: C49.2, H3.1
- new net: C46.1, H4.1
- new net: C47.1, H2.1
