File: PCB/EPS_KiCad_Design ruteo tobi/EPS_KiCad_Design/MCU.kicad_sch (KiCad schematic)
At the start: 26 parts, among them IC6 STM32L433CBT7, J2 FTSH-107-01-L-D-K, Y1 ABS07-LR-32.768KHZ-6-1-T, Y2 ABM3-8.000MHZ-D2Y-T

Commit message: Actualizacion del PCB
Parts:
- C15, C16: value 8.2pF -> 6.8pF
Changed lines of the file:
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@@
 			)
 		)
-		(property "Value" "8.2pF"
+		(property "Value" "6.8pF"
 			(at 40.64 55.626 90)
 			(effects
@@
 			)
 		)
-		(property "Value" "8.2pF"
+		(property "Value" "6.8pF"
 			(at 40.64 33.782 90)
 			(effects

Commit message: Cambio de conector
Conector header de 5 posiciones
Parts:
- removed J2: FTSH-107-01-L-D-K, FTSH-107-01-L-D-K_Footprint:FTSH-107-XX-YYY-D-K, symbol FTSH-107-01-L-D-K:FTSH-107-01-L-D-K
- added J2: Conn_01x05, TSM_Connector:TSM10501LSV, symbol Connector_Generic:Conn_01x05
Connections:
- net 3V3_1: now also J2.1 (Pin_1)
- net GND: now also J2.4 (Pin_4)
- net NRST: now also J2.5 (Pin_5)
- net PA13: now also J2.2 (Pin_2)
- net PA14: now also J2.3 (Pin_3)
- net PA2: no longer names the net of IC6.12 (PA2)
- net PA3: no longer names the net of IC6.13 (PA3)
- net PB3: no longer names the net of IC6.39 (PB3)
- no-connect marks 18 -> 17

Commit message: cambios en el ruteo
Changed lines of the file:
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@@
 	(wire
 		(pts
-			(xy 142.24 110.49) (xy 142.24 113.03)
+			(xy 142.24 110.49) (xy 142.24 116.84)
 		)
 		(stroke
@@
 	(wire
 		(pts
-			(xy 144.78 110.49) (xy 144.78 113.03)
+			(xy 144.78 110.49) (xy 144.78 116.84)
 		)
 		(stroke
@@
 	)
 	(label "PB10"
-		(at 142.24 113.03 270)
+		(at 142.24 116.84 270)
 		(effects
 			(font
@@
 	)
 	(label "PB11"
-		(at 144.78 113.03 270)
-		(effects
-			(font
+		(at 144.78 116.84 270)
+		(effects
+			(font
